File: pcb/ouderdag v2.kicad_pcb (KiCad board)
At the start: 2 copper layers, 101 x 50 mm, 18 parts, among them J1 Conn_01x05_Pin, J2 Conn_01x05_Pin, J3 Conn_01x05_Socket, J4 Conn_01x05_Socket, J5 Conn_01x06_Pin, SW1 SW_Push, U1 ATtiny85

Commit message: updated code and pcb
Parts:
- removed C1: C, Capacitor_THT:CP_Radial_D8.0mm_P3.50mm
- added J6: Conn_01x03_Pin, Connector_PinHeader_2.54mm:PinHeader_1x03_P2.54mm_Vertical, B.Cu at (77.5, 122.9)
- added Ref**: Val**, lib:Art, F.Cu at (126.0, 107.5)
- added Ref**: Val**, lib:Art, B.Cu at (117.5, 103.0)
- added SW2: SW-18020P, lib:SW-18020P, F.Cu at (105.0, 96.0)
- D1, D2, D3, D4, D5, D6, D7: footprint LED_THT:LED_D8.0mm -> LED_THT:LED_D10.0mm
- J1, J2: value Conn_01x05_Pin -> Conn_01x03_Pin; footprint Connector_PinHeader_2.54mm:PinHeader_1x05_P2.54mm_Vertical -> Connector_PinHeader_2.54mm:PinHeader_1x03_P2.54mm_Vertical
- J3, J4: value Conn_01x05_Socket -> Conn_01x03_Socket; footprint Connector_PinSocket_2.54mm:PinSocket_1x05_P2.54mm_Vertical -> Connector_PinSocket_2.54mm:PinSocket_1x03_P2.54mm_Vertical
- J5: value Conn_01x06_Pin -> Conn_01x03_Socket; footprint Connector_PinHeader_2.54mm:PinHeader_1x06_P2.54mm_Vertical -> Connector_PinSocket_2.54mm:PinSocket_1x03_P2.54mm_Vertical
- moved J5 46.6 mm to (128.5, 122.9)
- moved J1 23.0 mm to (52.1, 82.2), turned to 180 degrees
- moved J3 22.8 mm to (103.1, 82.2), turned to 0 degrees
- moved R2 17.7 mm to (82.0, 93.0), turned to 90 degrees
- moved J2 12.7 mm to (97.9, 82.2)
- moved J4 12.7 mm to (148.9, 82.2)
- moved BT1 8.33 mm to (135.0, 87.5), turned to 0 degrees
- moved SW1 3.50 mm to (68.9, 111.8)
- moved R1 2.94 mm to (68.0, 82.8), turned to -90 degrees
- moved U1 2.18 mm to (115.8, 89.8)
Connections:
- D1 pad 2: 2 -> PB1
- D2 pad 1: 2 -> PB1
- D3 pad 1: 3 -> PB2
- D5 pad 1: 3 -> PB2
- D6 pad 1: 2 -> PB1
- D7 pad 2: 2 -> PB1
- J1 pad 1: 1 -> PB0
- J1 pad 2: 2 -> PB1
- J1 pad 3: 3 -> PB2
- J2 pad 1: 1 -> PB0
- J2 pad 2: 2 -> PB1
- J2 pad 3: 3 -> PB2
- J3 pad 1: 1 -> PB0
- J3 pad 2: 2 -> PB1
- J3 pad 3: 3 -> PB2
- J4 pad 1: 1 -> PB0
- J4 pad 2: 2 -> PB1
- J4 pad 3: 3 -> PB2
- J5 pad 1: VCC -> GND
- J5 pad 2: 3 -> PB4
- J5 pad 3: 2 -> GND
- R1 pad 1: 3 -> PB2
- R2 pad 2: 1 -> PB0
- SW1 pad 2: 4 -> PB4
- U1 pad 1: RST -> PB5
- U1 pad 3: 4 -> PB4
- U1 pad 5: 1 -> PB0
- U1 pad 6: 2 -> PB1
- U1 pad 7: 3 -> PB2
Routing:
- net 1: track 181.9 -> 0.00 mm, vias 2 -> 0
- net 3: track 181.9 -> 0.00 mm, vias 1 -> 0
- net PB1: track 0.00 -> 172.4 mm, vias 0 -> 2
- net 2: track 169.2 -> 0.00 mm, vias 2 -> 0
- net 4: track 160.8 -> 0.00 mm, vias 1 -> 0
- net PB2: track 0.00 -> 139.5 mm, vias 0 -> 2
- net PB4: track 0.00 -> 107.8 mm, vias 0 -> 2
- net PB0: track 0.00 -> 105.5 mm, vias 0 -> 2
- net VCC: track 60.4 -> 17.2 mm
- net RST: track 15.2 -> 0.00 mm
- net GND: track 13.8 -> 0.00 mm, vias 24 -> 27
- net Net-(D4-A): track 16.6 -> 12.9 mm
- net Net-(D1-K): track 111.2 -> 112.1 mm
Other:
- outline, holes or cut-outs redrawn
- board text added: "CR2032"
- board text added: "Digi Dobbelsteen v1.0"
- board text added: "JLCJLCJLCJLC"
- board text removed: "Digi Dobbelsteen v0.1"

Commit message: change to generic ATtiny
PCB changes:
version 1.0 -> version 1.1
ATtiny85 -> ATtiny
mousebite trace FFF -> FBF
removed order number
Parts:
- R1, R2: value 220R -> 100R
- U1: value ATtiny85 -> ATtiny
Other:
- board text added: "Digi Dobbelsteen v1.1"
- board text removed: "Digi Dobbelsteen v1.0"
